Commit message: make it more readable

File: urdf/arm.urdf.xacro (robot description, xacro)
@@ -5,6 +5,5 @@
      For more information, please see http://wiki.ros.org/sw_urdf_exporter -->
 <xacro:property name="M_PI" value="3.1415926535897931" />
-  <link
-    name="base_link">
+  <link name="base_link">
     <!-- <inertial>
       <origin
@@ -29,8 +28,6 @@
           filename="package://arm_simulation/meshes/base_link.STL" />
       </geometry>
-      <material
-        name="">
-        <color
-          rgba="1 1 1 1" />
+      <material name="">
+        <color rgba="1 1 1 1" />
       </material>
     </visual>
@@ -45,12 +42,10 @@
     </collision>
   </link>
-  <link
-    name="link1">
+  <link name="link1">
     <inertial>
       <origin
         xyz="-6.2872E-18 7.6755E-18 0.035846"
         rpy="0 0 0" />
-      <mass
-        value="0.37205" />
+      <mass value="0.37205" />
       <inertia
         ixx="0.00018192"
@@ -69,8 +64,6 @@
           filename="package://arm_simulation/meshes/link1.STL" />
       </geometry>
-      <material
-        name="">
-        <color
-          rgba="1 1 1 1" />
+      <material name="">
+        <color rgba="1 1 1 1" />
       </material>
     </visual>
@@ -85,16 +78,11 @@
     </collision>
   </link>
-  <joint
-    name="joint1"
-    type="revolute">
+  <joint name="joint1" type="revolute">
     <origin
       xyz="0 0 0.074"
       rpy="0 0 0" />
-    <parent
-      link="base_link" />
-    <child
-      link="link1" />
-    <axis
-      xyz="0 0 1" />
+    <parent link="base_link" />
+    <child link="link1" />
+    <axis xyz="0 0 1" />
     <limit
       lower="-3.14"
@@ -103,12 +91,10 @@
       velocity="0" />
   </joint>
-  <link
-    name="link2">
+  <link name="link2">
     <inertial>
       <origin
         xyz="0.00027312 -6.8025E-07 0.11528"
         rpy="0 0 0" />
-      <mass
-        value="0.46302" />
+      <mass value="0.46302" />
       <inertia
         ixx="0.0050956"
@@ -127,8 +113,6 @@
           filename="package://arm_simulation/meshes/link2.STL" />
       </geometry>
-      <material
-        name="">
-        <color
-          rgba="1 1 1 1" />
+      <material name="">
+        <color rgba="1 1 1 1" />
       </material>
     </visual>
@@ -143,16 +127,11 @@
     </collision>
   </link>
-  <joint
-    name="joint2"
-    type="revolute">
+  <joint name="joint2" type="revolute">
     <origin
       xyz="-0.089 0.00023207 0.042"
       rpy="0.30054 -0.00073734 -0.00022852" />
-    <parent
-      link="link1" />
-    <child
-      link="link2" />
-    <axis
-      xyz="-1 0.0024907 0" />
+    <parent link="link1" />
+    <child link="link2" />
+    <axis xyz="-1 0.0024907 0" />
     <limit
       lower="-1.57"
@@ -161,12 +140,10 @@
       velocity="0" />
   </joint>
-  <link
-    name="link3">
+  <link name="link3">
     <inertial>
       <origin
         xyz="-0.0046535 0.020103 0.038177"
         rpy="0 0 0" />
-      <mass
-        value="0.06371" />
+      <mass value="0.06371" />
       <inertia
         ixx="9.6305E-05"
@@ -185,8 +162,6 @@
           filename="package://arm_simulation/meshes/link3.STL" />
       </geometry>
-      <material
-        name="">
-        <color
-          rgba="1 1 1 1" />
+      <material name="">
+        <color rgba="1 1 1 1" />
       </material>
     </visual>
@@ -201,16 +176,11 @@
     </collision>
   </link>
-  <joint
-    name="joint3"
-    type="revolute">
+  <joint name="joint3" type="revolute">
     <origin
       xyz="0.05725 -0.00014259 0.2789"
       rpy="0.79723 -0.0016401 3.1407" />
-    <parent
-      link="link2" />
-    <child
-      link="link3" />
-    <axis
-      xyz="1 -0.0022925 0" />
+    <parent link="link2" />
+    <child link="link3" />
+    <axis xyz="1 -0.0022925 0" />
     <limit
       lower="-1.57"
@@ -219,12 +189,10 @@
       velocity="0" />
   </joint>
-  <link
-    name="link4">
+  <link name="link4">
     <inertial>
       <origin
         xyz="0 -0.0016144 0.1471"
         rpy="0 0 0" />
-      <mass
-        value="0.41614" />
+      <mass value="0.41614" />
       <inertia
         ixx="0.0046604"
@@ -243,8 +211,6 @@
           filename="package://arm_simulation/meshes/link4.STL" />
       </geometry>
-      <material
-        name="">
-        <color
-          rgba="1 1 1 1" />
+      <material name="">
+        <color rgba="1 1 1 1" />
       </material>
     </visual>
@@ -259,16 +225,11 @@
     </collision>
   </link>
-  <joint
-    name="joint4"
-    type="revolute">
+  <joint name="joint4" type="revolute">
     <origin
       xyz="-0.031631 0.052087 0.064988"
       rpy="0.7035 1.3411 2.2852" />
-    <parent
-      link="link3" />
-    <child
-      link="link4" />
-    <axis
-      xyz="0 0 1" />
+    <parent link="link3" />
+    <child link="link4" />
+    <axis xyz="0 0 1" />
     <limit
       lower="-3.14"
@@ -277,12 +238,10 @@
       velocity="0" />
   </joint>
-  <link
-    name="link5">
+  <link name="link5">
     <inertial>
       <origin
         xyz="0.0026601 0.00039794 0.012151"
         rpy="0 0 0" />
-      <mass
-        value="0.030074" />
+      <mass value="0.030074" />
       <inertia
         ixx="1.6785E-05"
@@ -301,8 +260,6 @@
           filename="package://arm_simulation/meshes/link5.STL" />
       </geometry>
-      <material
-        name="">
-        <color
-          rgba="1 1 1 1" />
+      <material name="">
+        <color rgba="1 1 1 1" />
       </material>
     </visual>
@@ -317,16 +274,11 @@
     </collision>
   </link>
-  <joint
-    name="joint5"
-    type="revolute">
+  <joint name="joint5" type="revolute">
     <origin
       xyz="0 -0.034 0.2684"
       rpy="-0.0364343502514425 -0.00544912780563413 -1.71919063956753" />
-    <parent
-      link="link4" />
-    <child
-      link="link5" />
-    <axis
-      xyz="-0.999983629434664 0.00154627583027758 0.00550907376364283" />
+    <parent link="link4" />
+    <child link="link5" />
+    <axis xyz="-0.999983629434664 0.00154627583027758 0.00550907376364283" />
     <limit
       lower="-1.57"
@@ -335,3 +287,53 @@
       velocity="0" />
   </joint>
+  <!-- <transmission name="trans_joint1">
+      <type>transmission_interface/SimpleTransmission</type>
+      <joint name="joint1">
+          <hardwareInterface>hardware_interface/PositionJointInterface</hardwareInterface>
+      </joint>
+      <actuator name="joint1_motor">
+          <hardwareInterface>hardware_interface/PositionJointInterface</hardwareInterface>
+          <mechanicalReduction>1</mechanicalReduction>
+      </actuator>
+  </transmission>
+  <transmission name="trans_joint2">
+      <type>transmission_interface/SimpleTransmission</type>
+      <joint name="joint2">
+          <hardwareInterface>hardware_interface/PositionJointInterface</hardwareInterface>
+      </joint>
+      <actuator name="joint2_motor">
+          <hardwareInterface>hardware_interface/PositionJointInterface</hardwareInterface>
+          <mechanicalReduction>1</mechanicalReduction>
+      </actuator>
+  </transmission>
+  <transmission name="trans_joint3">
+      <type>transmission_interface/SimpleTransmission</type>
+      <joint name="joint3">
+          <hardwareInterface>hardware_interface/PositionJointInterface</hardwareInterface>
+      </joint>
+      <actuator name="joint3_motor">
+          <hardwareInterface>hardware_interface/PositionJointInterface</hardwareInterface>
+          <mechanicalReduction>1</mechanicalReduction>
+      </actuator>
+  </transmission>
+  <transmission name="trans_joint4">
+      <type>transmission_interface/SimpleTransmission</type>
+      <joint name="joint4">
+          <hardwareInterface>hardware_interface/PositionJointInterface</hardwareInterface>
+      </joint>
+      <actuator name="joint4_motor">
+          <hardwareInterface>hardware_interface/PositionJointInterface</hardwareInterface>
+          <mechanicalReduction>1</mechanicalReduction>
+      </actuator>
+  </transmission>
+  <transmission name="trans_joint5">
+      <type>transmission_interface/SimpleTransmission</type>
+      <joint name="joint5">
+          <hardwareInterface>hardware_interface/PositionJointInterface</hardwareInterface>
+      </joint>
+      <actuator name="joint5_motor">
+          <hardwareInterface>hardware_interface/PositionJointInterface</hardwareInterface>
+          <mechanicalReduction>1</mechanicalReduction>
+      </actuator>
+  </transmission> -->
 </robot>
