Commit message: changed dir to models; removed old rviz conf.

File: venus_description/urdf/venus.urdf.xacro (robot description, xacro)
@@ -20,5 +20,5 @@
   <xacro:venus parent="world" prefix="$(arg prefix)">
     <origin xyz="0 0 0" rpy="0 0 0" />
-  </xacro:rrbot>
+  </xacro:venus>
   <!-- <xacro:rrbot_ros2_control name="RRBot" prefix="$(arg prefix)" /> -->
 </robot>

File: venus_description/urdf/venus_description.urdf.xacro (robot description, xacro)
@@ -6,5 +6,5 @@
   <xacro:macro name="venus" params="parent prefix *origin">
   <!-- Constants for robot dimensions -->
-  <!-- TBD -->
+  <xacro:property name="pi_offset" value="0.001" />
   <joint name="${prefix}base_joint" type="fixed">
     <xacro:insert_block name="origin" />
@@ -15,13 +15,13 @@
   <link name="${prefix}base_link">
     <visual>
-      <origin xyz="0 0 0" rpy="pi/2 0 0" />
-      <geometry>
-        <mesh filename="package://arm_simulation/meshes/base_link.STL" />
-      </geometry>
-    </visual>
-    <collision>
-      <origin xyz="0 0 0" rpy="pi/2 0 0" />
-      <geometry>
-        <mesh filename="package://arm_simulation/meshes/base_link.STL" />
+      <origin xyz="0 0 0" rpy="${pi/2} 0 0" />
+      <geometry>
+        <mesh filename="package://venus_description/meshes/base_link.STL" />
+      </geometry>
+    </visual>
+    <collision>
+      <origin xyz="0 0 0" rpy="${pi/2} 0 0" />
+      <geometry>
+        <mesh filename="package://venus_description/meshes/base_link.STL" />
       </geometry>
     </collision>
@@ -49,12 +49,12 @@
       <origin xyz="0 0 0" rpy="0 0 0" />
       <geometry>
-        <mesh filename="package://arm_simulation/meshes/link1.STL" />
-      </geometry>
-    </visual>
-    <collision>
-      <origin xyz="0 0 0" rpy="0 0 0" />
-      <geometry>
-        <mesh
-          filename="package://arm_simulation/meshes/link1.STL" />
+        <mesh filename="package://venus_description/meshes/link1.STL" />
+      </geometry>
+    </visual>
+    <collision>
+      <origin xyz="0 0 0" rpy="0 0 0" />
+      <geometry>
+        <mesh
+          filename="package://venus_description/meshes/link1.STL" />
       </geometry>
     </collision>
@@ -73,5 +73,5 @@
     <origin xyz="-0.089 0.00023207 0.042" rpy="0.30054 -0.00073734 -0.00022852" />
     <axis xyz="-1 0.0024907 0" />
-    <limit lower="-pi/2" upper="pi/2" effort="2" velocity="5.5" />
+    <limit lower="-${pi/2}" upper="${pi/2}" effort="2" velocity="5.5" />
   </joint>
   <!-- Link2 -->
@@ -81,12 +81,12 @@
       <geometry>
         <mesh
-          filename="package://arm_simulation/meshes/link2.STL" />
-      </geometry>
-    </visual>
-    <collision>
-      <origin xyz="0 0 0" rpy="0 0 0" />
-      <geometry>
-        <mesh
-          filename="package://arm_simulation/meshes/link2.STL" />
+          filename="package://venus_description/meshes/link2.STL" />
+      </geometry>
+    </visual>
+    <collision>
+      <origin xyz="0 0 0" rpy="0 0 0" />
+      <geometry>
+        <mesh
+          filename="package://venus_description/meshes/link2.STL" />
       </geometry>
     </collision>
@@ -106,5 +106,5 @@
     <axis xyz="1 -0.0022925 0" />
     <limit
-      lower="-pi/2" upper="pi/2" effort="2" velocity="5.5" />
+      lower="-${pi/2}" upper="${pi/2}" effort="2" velocity="5.5" />
   </joint>
   <!-- Link3 -->
@@ -114,12 +114,12 @@
       <geometry>
         <mesh
-          filename="package://arm_simulation/meshes/link3.STL" />
-      </geometry>
-    </visual>
-    <collision>
-      <origin xyz="0 0 0" rpy="0 0 0" />
-      <geometry>
-        <mesh
-          filename="package://arm_simulation/meshes/link3.STL" />
+          filename="package://venus_description/meshes/link3.STL" />
+      </geometry>
+    </visual>
+    <collision>
+      <origin xyz="0 0 0" rpy="0 0 0" />
+      <geometry>
+        <mesh
+          filename="package://venus_description/meshes/link3.STL" />
       </geometry>
     </collision>
@@ -138,5 +138,5 @@
     <origin xyz="-0.031631 0.052087 0.064988" rpy="0.7035 1.3411 2.2852" />
     <axis xyz="0 0 1" />
-    <limit lower="-pi/2" upper="3.14" effort="2" velocity="5.5" />
+    <limit lower="-${pi}" upper="${pi}" effort="2" velocity="5.5" />
   </joint>
   <!-- Link4 -->
@@ -146,12 +146,12 @@
       <geometry>
         <mesh
-          filename="package://arm_simulation/meshes/link4.STL" />
-      </geometry>
-    </visual>
-    <collision>
-      <origin xyz="0 0 0" rpy="0 0 0" />
-      <geometry>
-        <mesh
-          filename="package://arm_simulation/meshes/link4.STL" />
+          filename="package://venus_description/meshes/link4.STL" />
+      </geometry>
+    </visual>
+    <collision>
+      <origin xyz="0 0 0" rpy="0 0 0" />
+      <geometry>
+        <mesh
+          filename="package://venus_description/meshes/link4.STL" />
       </geometry>
     </collision>
@@ -170,5 +170,5 @@
     <origin xyz="0 -0.034 0.2684" rpy="-0.0364343502514425 -0.00544912780563413 -1.71919063956753" />
     <axis xyz="-0.999983629434664 0.00154627583027758 0.00550907376364283" />
-    <limit lower="-pi/2" upper="1.57" effort="2" velocity="5.5" />
+    <limit lower="-${pi/2}" upper="${pi/2}" effort="2" velocity="5.5" />
   </joint>
   <!-- Link5 -->
@@ -178,12 +178,12 @@
       <geometry>
         <mesh
-          filename="package://arm_simulation/meshes/link5.STL" />
-      </geometry>
-    </visual>
-    <collision>
-      <origin xyz="0 0 0" rpy="0 0 0" />
-      <geometry>
-        <mesh
-          filename="package://arm_simulation/meshes/link5.STL" />
+          filename="package://venus_description/meshes/link5.STL" />
+      </geometry>
+    </visual>
+    <collision>
+      <origin xyz="0 0 0" rpy="0 0 0" />
+      <geometry>
+        <mesh
+          filename="package://venus_description/meshes/link5.STL" />
       </geometry>
     </collision>

Commit message: added color to the manipulator

File: venus_description/urdf/venus.urdf.xacro (robot description, xacro)
@@ -10,5 +10,5 @@
   <xacro:include filename="$(find venus_description)/urdf/venus_description.urdf.xacro" />
   <!-- Import Rviz colors -->
-  <!-- <xacro:include filename="$(find rrbot_description)/gazebo/rrbot.materials.xacro" /> -->
+  <xacro:include filename="$(find venus_description)/gazebo/venus.materials.xacro" />
   <!-- Import Venus ros2_control description -->
   <!-- <xacro:include filename="$(find rrbot_description)/ros2_control/rrbot.ros2_control.xacro" /> -->

File: venus_description/urdf/venus_description.urdf.xacro (robot description, xacro)
@@ -19,4 +19,5 @@
         <mesh filename="package://venus_description/meshes/base_link.STL" />
       </geometry>
+      <material name="grey"/>
     </visual>
     <collision>
@@ -51,4 +52,5 @@
         <mesh filename="package://venus_description/meshes/link1.STL" />
       </geometry>
+      <material name="grey"/>
     </visual>
     <collision>
@@ -83,4 +85,5 @@
           filename="package://venus_description/meshes/link2.STL" />
       </geometry>
+      <material name="grey"/>
     </visual>
     <collision>
@@ -116,4 +119,5 @@
           filename="package://venus_description/meshes/link3.STL" />
       </geometry>
+      <material name="grey"/>
     </visual>
     <collision>
@@ -148,4 +152,5 @@
           filename="package://venus_description/meshes/link4.STL" />
       </geometry>
+      <material name="grey"/>
     </visual>
     <collision>
@@ -180,4 +185,5 @@
           filename="package://venus_description/meshes/link5.STL" />
       </geometry>
+      <material name="grey"/>
     </visual>
     <collision>
