Commit message: Fixed yaml error when launching

File: venus_description/urdf/venus_description.urdf.xacro (robot description, xacro)
@@ -1,10 +1,10 @@
 <?xml version="1.0" encoding="utf-8"?>
 <robot xmlns:xacro="http://www.ros.org/wiki/xacro">
-<!-- This URDF was automatically created by SolidWorks to URDF Exporter! Originally created by Stephen Brawner (brawner@gmail.com)
-     Commit Version: 1.6.0-1-g15f4949  Build Version: 1.6.7594.29634
-     For more information, please see http://wiki.ros.org/sw_urdf_exporter -->
+<!-- This URDF was automatically created by SolidWorks to URDF Exporter!
+  Originally created by Stephen Brawner (brawner@gmail.com)
+  For more information, please see http://wiki.ros.org/sw_urdf_exporter -->
   <xacro:macro name="venus" params="parent prefix *origin">
   <!-- Constants for robot dimensions -->
-  <xacro:property name="pi_offset" value="0.001" />
+  <!-- <xacro:property name="pi_offset" value="0.001" /> -->
   <joint name="${prefix}base_joint" type="fixed">
     <xacro:insert_block name="origin" />

Commit message: Adjust the pose of the manipulator to match the calibration mark

File: venus_description/urdf/venus_description.urdf.xacro (robot description, xacro)
@@ -73,6 +73,7 @@
     <parent link="${prefix}link1" />
     <child link="${prefix}link2" />
-    <origin xyz="-0.089 0.00023207 0.042" rpy="0.30054 -0.00073734 -0.00022852" />
-    <axis xyz="-1 0.0024907 0" />
+    <!-- <origin xyz="-0.089 0 0.042" rpy="0.30054 0 0" /> -->
+    <origin xyz="-0.089 0 0.042" rpy="0 0 0" />
+    <axis xyz="-1 0 0" />
     <limit lower="-${pi/2}" upper="${pi/2}" effort="2" velocity="5.5" />
   </joint>
@@ -106,6 +107,7 @@
     <parent link="${prefix}link2" />
     <child link="${prefix}link3" />
-    <origin xyz="0.05725 -0.00014259 0.2789" rpy="0.79723 -0.0016401 3.1407" />
-    <axis xyz="1 -0.0022925 0" />
+    <!-- <origin xyz="0.05725 -0.00014259 0.2789" rpy="0.79723 -0.0016401 3.1407" /> -->
+    <origin xyz="0.05725 0 0.2789" rpy="0 0 ${pi}" />
+    <axis xyz="1 0 0" />
     <limit
       lower="-${pi/2}" upper="${pi/2}" effort="2" velocity="5.5" />
@@ -140,5 +142,6 @@
     <parent link="${prefix}link3" />
     <child link="${prefix}link4" />
-    <origin xyz="-0.031631 0.052087 0.064988" rpy="0.7035 1.3411 2.2852" />
+    <!-- <origin xyz="-0.031631 0.052087 0.064988" rpy="0.7035 1.3411 2.2852" /> -->
+    <origin xyz="-0.031631 0.052087 0.064988" rpy="${-80*pi/180} 0 0" />
     <axis xyz="0 0 1" />
     <limit lower="-${pi}" upper="${pi}" effort="2" velocity="5.5" />
@@ -147,5 +150,5 @@
   <link name="${prefix}link4">
     <visual>
-      <origin xyz="0 0 0" rpy="0 0 0" />
+      <origin xyz="0 0 0" rpy="0 0 ${pi/2}" />
       <geometry>
         <mesh
@@ -155,5 +158,5 @@
     </visual>
     <collision>
-      <origin xyz="0 0 0" rpy="0 0 0" />
+      <origin xyz="0 0 0" rpy="0 0 ${pi/2}" />
       <geometry>
         <mesh
@@ -173,6 +176,7 @@
     <parent link="${prefix}link4" />
     <child link="${prefix}link5" />
-    <origin xyz="0 -0.034 0.2684" rpy="-0.0364343502514425 -0.00544912780563413 -1.71919063956753" />
-    <axis xyz="-0.999983629434664 0.00154627583027758 0.00550907376364283" />
+    <!-- <origin xyz="0 -0.034 0.2684" rpy="-0.0364343502514425 -0.00544912780563413 -1.71919063956753" /> -->
+    <origin xyz="0 0 0.2684" rpy="0 0 0" />
+    <axis xyz="-1 0 0" />
     <limit lower="-${pi/2}" upper="${pi/2}" effort="2" velocity="5.5" />
   </joint>
@@ -180,5 +184,5 @@
   <link name="${prefix}link5">
     <visual>
-      <origin xyz="0 0 0" rpy="0 0 0" />
+      <origin xyz="0.033 0 0" rpy="0 0 -0.15" />
       <geometry>
         <mesh
@@ -188,5 +192,5 @@
     </visual>
     <collision>
-      <origin xyz="0 0 0" rpy="0 0 0" />
+      <origin xyz="0.033 0 0" rpy="0 0 -0.15" />
       <geometry>
         <mesh

Commit message: changed joint axis direction to match sign convention

File: venus_description/urdf/venus_description.urdf.xacro (robot description, xacro)
@@ -45,5 +45,5 @@
     <child link="${prefix}link1" />
     <origin xyz="0 0 0.074" rpy="0 0 0" />
-    <axis xyz="0 0 1" />
+    <axis xyz="0 0 -1" />
     <limit effort="2" velocity="5.5" />
   </joint>
@@ -112,5 +112,5 @@
     <!-- <origin xyz="0.05725 -0.00014259 0.2789" rpy="0.79723 -0.0016401 3.1407" /> -->
     <origin xyz="0.05725 0 0.2789" rpy="0 0 ${pi}" />
-    <axis xyz="1 0 0" />
+    <axis xyz="-1 0 0" />
     <limit
       lower="-${pi/2}" upper="${pi/2}" effort="2" velocity="5.5" />
@@ -147,5 +147,5 @@
     <!-- <origin xyz="-0.031631 0.052087 0.064988" rpy="0.7035 1.3411 2.2852" /> -->
     <origin xyz="-0.031631 0.052087 0.064988" rpy="${-80*pi/180} 0 0" />
-    <axis xyz="0 0 1" />
+    <axis xyz="0 0 -1" />
     <limit lower="-${pi}" upper="${pi}" effort="2" velocity="5.5" />
   </joint>

Commit message: deleted transmissions

File: venus_description/urdf/venus_description.urdf.xacro (robot description, xacro)
@@ -211,53 +211,3 @@
   </link>
   </xacro:macro>
-  <!-- <transmission name="trans_joint1">
-      <type>transmission_interface/SimpleTransmission</type>
-      <joint name="joint1">
-          <hardwareInterface>hardware_interface/PositionJointInterface</hardwareInterface>
-      </joint>
-      <actuator name="joint1_motor">
-          <hardwareInterface>hardware_interface/PositionJointInterface</hardwareInterface>
-          <mechanicalReduction>1</mechanicalReduction>
-      </actuator>
-  </transmission>
-  <transmission name="trans_joint2">
-      <type>transmission_interface/SimpleTransmission</type>
-      <joint name="joint2">
-          <hardwareInterface>hardware_interface/PositionJointInterface</hardwareInterface>
-      </joint>
-      <actuator name="joint2_motor">
-          <hardwareInterface>hardware_interface/PositionJointInterface</hardwareInterface>
-          <mechanicalReduction>1</mechanicalReduction>
-      </actuator>
-  </transmission>
-  <transmission name="trans_joint3">
-      <type>transmission_interface/SimpleTransmission</type>
-      <joint name="joint3">
-          <hardwareInterface>hardware_interface/PositionJointInterface</hardwareInterface>
-      </joint>
-      <actuator name="joint3_motor">
-          <hardwareInterface>hardware_interface/PositionJointInterface</hardwareInterface>
-          <mechanicalReduction>1</mechanicalReduction>
-      </actuator>
-  </transmission>
-  <transmission name="trans_joint4">
-      <type>transmission_interface/SimpleTransmission</type>
-      <joint name="joint4">
-          <hardwareInterface>hardware_interface/PositionJointInterface</hardwareInterface>
-      </joint>
-      <actuator name="joint4_motor">
-          <hardwareInterface>hardware_interface/PositionJointInterface</hardwareInterface>
-          <mechanicalReduction>1</mechanicalReduction>
-      </actuator>
-  </transmission>
-  <transmission name="trans_joint5">
-      <type>transmission_interface/SimpleTransmission</type>
-      <joint name="joint5">
-          <hardwareInterface>hardware_interface/PositionJointInterface</hardwareInterface>
-      </joint>
-      <actuator name="joint5_motor">
-          <hardwareInterface>hardware_interface/PositionJointInterface</hardwareInterface>
-          <mechanicalReduction>1</mechanicalReduction>
-      </actuator>
-  </transmission> -->
 </robot>
