Commit message: Modified file names to make them more meaningful

File: venus_description/ros2_control/venus.ros2_control.xacro (robot description, xacro)
@@ -1,16 +1,31 @@
 <?xml version="1.0"?>
 <robot xmlns:xacro="http://www.ros.org/wiki/xacro">
-  <xacro:macro name="venus_ros2_control" params="name prefix">
+  <xacro:macro name="venus_control" params="name prefix
+  use_sim:=^|false
+  use_fake_hardware:=^|true fake_sensor_commands:=^|false">
     <ros2_control name="${name}" type="system">
-      <hardware>
-        <plugin>venus_hardware/VenusSystemPositionOnlyHardware</plugin>
-        <param name="example_param_hw_start_duration_sec">0</param>
-        <param name="example_param_hw_stop_duration_sec">3.0</param>
-        <param name="example_param_hw_slowdown">100</param>
-      </hardware>
+      <!-- <xacro:if value="$(arg use_sim)">
+        <hardware>
+          <plugin>gazebo_ros2_control/GazeboSystem</plugin>
+        </hardware>
+      </xacro:if> -->
+      <xacro:unless value="$(arg use_sim)">
+        <hardware>
+          <xacro:if value="${use_fake_hardware}">
+            <plugin>fake_components/GenericSystem</plugin>
+            <param name="fake_sensor_commands">${fake_sensor_commands}</param>
+            <param name="state_following_offset">0.0</param>
+          </xacro:if>
+          <xacro:unless value="${use_fake_hardware}">
+            <plugin>venus_hardware/VenusSystemPositionOnlyHardware</plugin>
+            <param name="example_param_hw_start_duration_sec">2.0</param>
+            <param name="example_param_hw_stop_duration_sec">3.0</param>
+          </xacro:unless>
+        </hardware>
+      </xacro:unless>
       <joint name="${prefix}joint1">
         <command_interface name="position">
-          <param name="min">-1</param>
-          <param name="max">1</param>
+          <param name="min">{-2*pi}</param>
+          <param name="max">{2*pi}</param>
         </command_interface>
         <state_interface name="position"/>
@@ -18,6 +33,6 @@
       <joint name="${prefix}joint2">
         <command_interface name="position">
-          <param name="min">-1</param>
-          <param name="max">1</param>
+          <param name="min">{-pi/2}</param>
+          <param name="max">{pi/2}</param>
         </command_interface>
         <state_interface name="position"/>
@@ -25,6 +40,6 @@
       <joint name="${prefix}joint3">
         <command_interface name="position">
-          <param name="min">-1</param>
-          <param name="max">1</param>
+          <param name="min">{-pi/2}</param>
+          <param name="max">{pi/2}</param>
         </command_interface>
         <state_interface name="position"/>
@@ -32,6 +47,6 @@
       <joint name="${prefix}joint4">
         <command_interface name="position">
-          <param name="min">-1</param>
-          <param name="max">1</param>
+          <param name="min">{-2*pi}</param>
+          <param name="max">{2*pi}</param>
         </command_interface>
         <state_interface name="position"/>
@@ -39,6 +54,6 @@
       <joint name="${prefix}joint5">
         <command_interface name="position">
-          <param name="min">-1</param>
-          <param name="max">1</param>
+          <param name="min">{-pi/2}</param>
+          <param name="max">{pi/2}</param>
         </command_interface>
         <state_interface name="position"/>

File: venus_description/urdf/venus.urdf.xacro (robot description, xacro)
@@ -11,6 +11,4 @@
   <!-- Import Rviz colors -->
   <xacro:include filename="$(find venus_description)/gazebo/venus.materials.xacro" />
-  <!-- Import Venus ros2_control description -->
-  <xacro:include filename="$(find venus_description)/ros2_control/venus.ros2_control.xacro" />
   <!-- Used for fixing robot -->
   <link name="world"/>
@@ -21,4 +19,3 @@
     <origin xyz="0 0 0" rpy="0 0 0" />
   </xacro:venus>
-  <xacro:venus_ros2_control name="Venus" prefix="$(arg prefix)" />
 </robot>

File: venus_description/urdf/venus_description.urdf.xacro (robot description, xacro)
@@ -1,10 +1,13 @@
 <?xml version="1.0" encoding="utf-8"?>
 <robot xmlns:xacro="http://www.ros.org/wiki/xacro">
-<!-- This URDF was automatically created by SolidWorks to URDF Exporter!
-  Originally created by Stephen Brawner (brawner@gmail.com)
-  For more information, please see http://wiki.ros.org/sw_urdf_exporter -->
+<!--
+  Base xacro macro.
+  NOTE this is NOT a URDF. It cannot directly be loaded by consumers
+  expecting a flattened '.urdf' file. XACRO is a macro language used in URDF
+  to better describe the model. See the XACRO instruction in ROS Wiki.
+  A xacro file must be processed by the xacro command to parse the model.
+-->
   <xacro:macro name="venus" params="parent prefix *origin">
   <!-- Constants for robot dimensions -->
-  <!-- <xacro:property name="pi_offset" value="0.001" /> -->
   <joint name="${prefix}base_joint" type="fixed">
     <xacro:insert_block name="origin" />

File: venus_description/urdf/venus_with_controller.urdf.xacro (robot description, xacro)
@@ -11,5 +11,4 @@
   <xacro:arg name="fake_sensor_commands" default="false" />
   <xacro:arg name="prefix" default="" />
-  <xacro:arg name="slowdown" default="2.0" />
   <!-- Import Venus macro -->
   <xacro:include filename="$(find venus_description)/urdf/venus_description.urdf.xacro" />
@@ -19,5 +18,5 @@
   <xacro:include filename="$(find venus_description)/gazebo/venus.materials.xacro" />
   <!-- Import Venus ros2_control description -->
-  <xacro:include filename="$(find venus_description)/ros2_control/venus_system_position_only.ros2_control.xacro" />
+  <xacro:include filename="$(find venus_description)/ros2_control/venus.ros2_control.xacro" />
   <!-- Used for fixing robot -->
   <link name="world"/>
@@ -29,8 +28,7 @@
   </xacro:venus>
   <!-- <xacro:rrbot_gazebo prefix="$(arg prefix)" /> -->
-  <xacro:venus_system_position_only
+  <xacro:venus_control
     name="VenusSystemPositionOnly" prefix="$(arg prefix)"
     use_fake_hardware="$(arg use_fake_hardware)"
-    fake_sensor_commands="$(arg fake_sensor_commands)"
-    slowdown="$(arg slowdown)" />
+    fake_sensor_commands="$(arg fake_sensor_commands)" />
 </robot>
